Commit message: 机械臂第一版添加

File: my_robot_description/urdf/common/inertia_macros.xacro (robot description, xacro)
@@ -19,3 +19,13 @@
         </inertial>
     </xacro:macro>
+    <!-- 添加长方体惯性宏 -->
+    <xacro:macro name="box_inertia" params="m x y z">
+        <inertial>
+            <origin xyz="0 0 0" rpy="0 0 0" />
+            <mass value="${m}" />
+            <inertia ixx="${(m/12) * (y*y + z*z)}" ixy="0" ixz="0"
+                     iyy="${(m/12) * (x*x + z*z)}" iyz="0"
+                     izz="${(m/12) * (x*x + y*y)}" />
+        </inertial>
+    </xacro:macro>
 </robot>

File: my_robot_description/urdf/test_base.xacro (robot description, xacro)
@@ -4,5 +4,9 @@
     <xacro:include filename="base/mobile_base.xacro" />
     <xacro:include filename="base/mobile_base_gazebo.xacro" />
+    <xacro:include filename="arm/simple_arm.xacro" />
+    <xacro:include filename="arm/simple_arm_gazebo.xacro" />
     <xacro:mobile_base />
     <xacro:mobile_base_gazebo_plugin />
+    <xacro:simple_arm prefix="arm_" />
+    <xacro:simple_arm_gazebo_plugin prefix="arm_" />
 </robot>
