Commit message: Add files via upload

File: my_robot_description/urdf/sensors/lidar.xacro (robot description, xacro)
@@ -6,5 +6,5 @@
         <origin xyz="0 0 0" rpy="0 0 0"/>
         <geometry>
-          <cylinder length="0.05" radius="0.05"/>
+          <cylinder length="0.01" radius="0.01"/>
         </geometry>
         <material name="black"/>
@@ -13,5 +13,5 @@
         <origin xyz="0 0 0" rpy="0 0 0"/>
         <geometry>
-          <cylinder length="0.05" radius="0.05"/>
+          <cylinder length="0.01" radius="0.01"/>
         </geometry>
       </collision>
@@ -21,5 +21,5 @@
       <parent link="base_link"/>
       <child link="${prefix}_link"/>
-      <origin xyz="0.20 0 0.01" rpy="0 0 0"/>
+      <origin xyz="0.15 0 0.01" rpy="0 0 0"/>
     </joint>
     <gazebo reference="${prefix}_link">
@@ -40,5 +40,5 @@
           </scan>
           <range>
-            <min>0.1</min>
+            <min>0.2</min>
             <max>10.0</max>
             <resolution>0.01</resolution>
