Commit message: new version

File: my_robot_description/urdf/base/mobile_base.xacro (robot description, xacro)
@@ -1,104 +1,118 @@
 <?xml version="1.0"?>
 <robot xmlns:xacro="http://www.ros.org/wiki/xacro">
-    <xacro:macro name="mobile_base">
-        <xacro:property name="chassis_radius" value="0.14" />
-        <xacro:property name="chassis_height" value="0.12" />
-        <xacro:property name="chassis_mass" value="10.0" />
-        <xacro:property name="wheel_radius" value="0.04" />
-        <xacro:property name="wheel_width" value="0.02" />
-        <xacro:property name="wheel_offset_y" value="0.13" />
-        <xacro:property name="caster_radius" value="0.02" />
-        <xacro:property name="caster_offset_x" value="0.10" />
-        <link name="base_footprint" >
-            <inertial>
-                <mass value="0.001"/>
-                <origin xyz="0 0 0"/>
-                <inertia ixx="0.0001" ixy="0.0" ixz="0.0"
-                         iyy="0.0001" iyz="0.0"
-                         izz="0.0001"/>
-            </inertial>
-        </link>
-        <joint name="base_joint" type="fixed">
-            <parent link="base_footprint" />
-            <child link="base_link" />
-            <origin xyz="0 0 ${wheel_radius}" rpy="0 0 0" />
-        </joint>
-        <link name="base_link">
-            <visual>
-                <origin xyz="0 0 ${chassis_height/2}" rpy="0 0 0" />
-                <geometry>
-                    <cylinder radius="${chassis_radius}" length="${chassis_height}" />
-                </geometry>
-                <material name="blue" />
-            </visual>
-            <collision>
-                <origin xyz="0 0 ${chassis_height/2}" rpy="0 0 0" />
-                <geometry>
-                    <cylinder radius="${chassis_radius}" length="${chassis_height}" />
-                </geometry>
-            </collision>
-            <xacro:cylinder_inertia m="${chassis_mass}" r="${chassis_radius}" h="${chassis_height}" />
-        </link>
-        <xacro:macro name="wheel" params="prefix y_reflect">
-            <link name="${prefix}_wheel_link">
-                <visual>
-                    <origin xyz="0 0 0" rpy="${pi/2} 0 0" />
-                    <geometry>
-                        <cylinder radius="${wheel_radius}" length="${wheel_width}" />
-                    </geometry>
-                    <material name="black" />
-                </visual>
-                <collision>
-                    <origin xyz="0 0 0" rpy="${pi/2} 0 0" />
-                    <geometry>
-                        <cylinder radius="${wheel_radius}" length="${wheel_width}" />
-                    </geometry>
-                </collision>
-                <xacro:cylinder_inertia m="0.5" r="${wheel_radius}" h="${wheel_width}" />
-            </link>
-            <joint name="${prefix}_wheel_joint" type="continuous">
-                <parent link="base_link" />
-                <child link="${prefix}_wheel_link" />
-                <origin xyz="0 ${y_reflect * wheel_offset_y} 0" rpy="0 0 0" />
-                <axis xyz="0 1 0" />
-            </joint>
-            <gazebo reference="${prefix}_wheel_link">
-                <mu1>2.0</mu1>
-                <mu2>2.0</mu2>
-                <kp>1000000.0</kp>
-                <kd>100.0</kd>
-                <material>Gazebo/Black</material>
-            </gazebo>
-        </xacro:macro>
-        <xacro:wheel prefix="left" y_reflect="1" />
-        <xacro:wheel prefix="right" y_reflect="-1" />
-        <xacro:macro name="caster_wheel" params="prefix x_reflect">
-            <link name="${prefix}_caster_wheel">
-                <visual>
-                    <geometry>
-                        <sphere radius="${caster_radius}" />
-                    </geometry>
-                    <material name="black" />
-                </visual>
-                <collision>
-                    <geometry>
-                        <sphere radius="${caster_radius}" />
-                    </geometry>
-                </collision>
-                <xacro:sphere_inertia m="0.1" r="${caster_radius}" />
-            </link>
-            <joint name="${prefix}_caster_joint" type="fixed">
-                <parent link="base_link" />
-                <child link="${prefix}_caster_wheel" />
-                <origin xyz="${x_reflect * caster_offset_x} 0 ${caster_radius - wheel_radius}" rpy="0 0 0" />
-            </joint>
-            <gazebo reference="${prefix}_caster_wheel">
-                <mu1>0.001</mu1>
-                <mu2>0.001</mu2>
-                <material>Gazebo/Black</material>
-            </gazebo>
-        </xacro:macro>
-        <xacro:caster_wheel prefix="front" x_reflect="1" />
-        <xacro:caster_wheel prefix="back" x_reflect="-1" />
+  <xacro:macro name="mobile_base">
+    <!-- ========== 参数 ========== -->
+    <xacro:property name="chassis_radius" value="0.14" />
+    <xacro:property name="chassis_height" value="0.12" />
+    <xacro:property name="chassis_mass" value="10.0" />
+    <xacro:property name="wheel_radius" value="0.04" />
+    <xacro:property name="wheel_width" value="0.02" />
+    <xacro:property name="wheel_offset_y" value="0.13" />
+    <xacro:property name="caster_radius" value="0.02" />
+    <xacro:property name="caster_offset_x" value="0.10" />
+    <!-- ========== base footprint ========== -->
+    <link name="base_footprint">
+      <inertial>
+        <mass value="0.001"/>
+        <origin xyz="0 0 0"/>
+        <inertia ixx="0.0001" ixy="0" ixz="0"
+                 iyy="0.0001" iyz="0"
+                 izz="0.0001"/>
+      </inertial>
+    </link>
+    <joint name="base_joint" type="fixed">
+      <parent link="base_footprint"/>
+      <child link="base_link"/>
+      <origin xyz="0 0 ${wheel_radius}" rpy="0 0 0"/>
+    </joint>
+    <!-- ========== base link ========== -->
+    <link name="base_link">
+      <visual>
+        <origin xyz="0 0 ${chassis_height/2}" rpy="0 0 0"/>
+        <geometry>
+          <cylinder radius="${chassis_radius}" length="${chassis_height}"/>
+        </geometry>
+        <material name="blue"/>
+      </visual>
+      <collision>
+        <origin xyz="0 0 ${chassis_height/2}" rpy="0 0 0"/>
+        <geometry>
+          <cylinder radius="${chassis_radius}" length="${chassis_height}"/>
+        </geometry>
+      </collision>
+      <xacro:cylinder_inertia
+        m="${chassis_mass}"
+        r="${chassis_radius}"
+        h="${chassis_height}"/>
+    </link>
+    <!-- ========== 轮子宏 ========== -->
+    <xacro:macro name="wheel" params="prefix y_reflect">
+      <link name="${prefix}_wheel_link">
+        <visual>
+          <!-- 轮子横放 -->
+          <origin xyz="0 0 0" rpy="${pi/2} 0 0"/>
+          <geometry>
+            <cylinder radius="${wheel_radius}" length="${wheel_width}"/>
+          </geometry>
+          <material name="black"/>
+        </visual>
+        <collision>
+          <origin xyz="0 0 0" rpy="${pi/2} 0 0"/>
+          <geometry>
+            <cylinder radius="${wheel_radius}" length="${wheel_width}"/>
+          </geometry>
+        </collision>
+        <xacro:cylinder_inertia
+          m="0.5"
+          r="${wheel_radius}"
+          h="${wheel_width}"/>
+      </link>
+      <joint name="${prefix}_wheel_joint" type="continuous">
+        <parent link="base_link"/>
+        <child link="${prefix}_wheel_link"/>
+        <origin xyz="0 ${y_reflect * wheel_offset_y} 0" rpy="0 0 0"/>
+        <axis xyz="0 1 0"/>
+      </joint>
+      <gazebo reference="${prefix}_wheel_link">
+        <mu1>2.0</mu1>
+        <mu2>2.0</mu2>
+        <kp>1000000.0</kp>
+        <kd>100.0</kd>
+        <gravity>true</gravity>
+        <self_collide>false</self_collide>
+      </gazebo>
     </xacro:macro>
+    <!-- 左右轮 -->
+    <xacro:wheel prefix="left"  y_reflect="1"/>
+    <xacro:wheel prefix="right" y_reflect="-1"/>
+    <!-- ========== 脚轮 ========== -->
+    <xacro:macro name="caster_wheel" params="prefix x_reflect">
+      <link name="${prefix}_caster_wheel">
+        <visual>
+          <geometry>
+            <sphere radius="${caster_radius}"/>
+          </geometry>
+          <material name="black"/>
+        </visual>
+        <collision>
+          <geometry>
+            <sphere radius="${caster_radius}"/>
+          </geometry>
+        </collision>
+        <xacro:sphere_inertia m="0.1" r="${caster_radius}"/>
+      </link>
+      <joint name="${prefix}_caster_joint" type="fixed">
+        <parent link="base_link"/>
+        <child link="${prefix}_caster_wheel"/>
+        <origin xyz="${x_reflect * caster_offset_x} 0 ${caster_radius - wheel_radius}" rpy="0 0 0"/>
+      </joint>
+      <gazebo reference="${prefix}_caster_wheel">
+        <mu1>0.001</mu1>
+        <mu2>0.001</mu2>
+        <gravity>true</gravity>
+      </gazebo>
+    </xacro:macro>
+    <xacro:caster_wheel prefix="front" x_reflect="1"/>
+    <xacro:caster_wheel prefix="back"  x_reflect="-1"/>
+  </xacro:macro>
 </robot>

File: my_robot_description/urdf/base/mobile_base_gazebo.xacro (robot description, xacro)
@@ -1,36 +1,39 @@
 <?xml version="1.0"?>
 <robot xmlns:xacro="http://www.ros.org/wiki/xacro">
-    <xacro:macro name="mobile_base_gazebo_plugin">
-        <gazebo>
-            <plugin filename="libignition-gazebo-diff-drive-system.so"
-                    name="ignition::gazebo::systems::DiffDrive">
-                <left_joint>left_wheel_joint</left_joint>
-                <right_joint>right_wheel_joint</right_joint>
-                <wheel_separation>0.26</wheel_separation>
-                <wheel_radius>0.04</wheel_radius>
-                <max_linear_acceleration>1</max_linear_acceleration>
-                <min_linear_acceleration>-1</min_linear_acceleration>
-                <max_angular_acceleration>2</max_angular_acceleration>
-                <min_angular_acceleration>-2</min_angular_acceleration>
-                <max_linear_velocity>0.5</max_linear_velocity>
-                <min_linear_velocity>-0.5</min_linear_velocity>
-                <max_angular_velocity>1</max_angular_velocity>
-                <min_angular_velocity>-1</min_angular_velocity>
-                <topic>cmd_vel</topic>
-                <odom_topic>odom</odom_topic>
-                <tf_topic>tf</tf_topic>
-                <frame_id>odom</frame_id>
-                <child_frame_id>base_footprint</child_frame_id>
-                <odom_publish_frequency>30</odom_publish_frequency>
-            </plugin>
-            <plugin filename="libignition-gazebo-joint-state-publisher-system.so"
-                    name="ignition::gazebo::systems::JointStatePublisher">
-                <topic>joint_states</topic>
-            </plugin>
-            <plugin filename="libignition-gazebo-sensors-system.so"
-                    name="ignition::gazebo::systems::Sensors">
-                <render_engine>ogre2</render_engine>
-            </plugin>
-        </gazebo>
-    </xacro:macro>
+  <xacro:macro name="mobile_base_gazebo_plugin">
+    <gazebo>
+      <!-- ========== Diff Drive ========== -->
+      <plugin
+        filename="libgz-sim-diff-drive-system.so"
+        name="gz::sim::systems::DiffDrive">
+        <left_joint>left_wheel_joint</left_joint>
+        <right_joint>right_wheel_joint</right_joint>
+        <wheel_separation>0.26</wheel_separation>
+        <wheel_radius>0.04</wheel_radius>
+        <max_linear_velocity>0.5</max_linear_velocity>
+        <min_linear_velocity>-0.5</min_linear_velocity>
+        <max_angular_velocity>1.0</max_angular_velocity>
+        <min_angular_velocity>-1.0</min_angular_velocity>
+        <!-- ★ 使用绝对 topic -->
+        <topic>/cmd_vel</topic>
+        <odom_topic>/odom</odom_topic>
+        <tf_topic>/tf</tf_topic>
+        <frame_id>odom</frame_id>
+        <child_frame_id>base_link</child_frame_id>
+        <odom_publish_frequency>30</odom_publish_frequency>
+      </plugin>
+      <!-- ========== Joint States ========== -->
+      <plugin
+        filename="libgz-sim-joint-state-publisher-system.so"
+        name="gz::sim::systems::JointStatePublisher">
+        <topic>/joint_states</topic>
+      </plugin>
+      <!-- ========== Sensors ========== -->
+      <plugin
+        filename="libgz-sim-sensors-system.so"
+        name="gz::sim::systems::Sensors">
+        <render_engine>ogre2</render_engine>
+      </plugin>
+    </gazebo>
+  </xacro:macro>
 </robot>

Commit message: Add files via upload

File: my_robot_description/urdf/base/mobile_base.xacro (robot description, xacro)
@@ -63,9 +63,17 @@
           </geometry>
         </collision>
-        <xacro:cylinder_inertia
-          m="0.5"
-          r="${wheel_radius}"
-          h="${wheel_width}"/>
+        <!-- ★★★ 关键修改：惯性矩阵的轴要与轮一致 ★★★ -->
+        <inertial>
+          <origin xyz="0 0 0" rpy="${pi/2} 0 0"/>
+          <mass value="0.5"/>
+          <inertia
+            ixx="${(0.5/12) * (3*wheel_radius*wheel_radius + wheel_width*wheel_width)}"
+            ixy="0" ixz="0"
+            iyy="${(0.5/12) * (3*wheel_radius*wheel_radius + wheel_width*wheel_width)}"
+            iyz="0"
+            izz="${(0.5/2) * (wheel_radius*wheel_radius)}"/>
+        </inertial>
       </link>
+      <!-- ★★★ 关键修改：axis 改为   轴 ★★★ -->
       <joint name="${prefix}_wheel_joint" type="continuous">
         <parent link="base_link"/>
@@ -73,8 +81,9 @@
         <origin xyz="0 ${y_reflect * wheel_offset_y} 0" rpy="0 0 0"/>
         <axis xyz="0 1 0"/>
+        <limit effort="0.2" velocity="20.0"/>
       </joint>
       <gazebo reference="${prefix}_wheel_link">
-        <mu1>2.0</mu1>
-        <mu2>2.0</mu2>
+        <mu1>1.0</mu1>
+        <mu2>1.0</mu2>
         <kp>1000000.0</kp>
         <kd>100.0</kd>

File: my_robot_description/urdf/base/mobile_base_gazebo.xacro (robot description, xacro)
@@ -2,38 +2,35 @@
 <robot xmlns:xacro="http://www.ros.org/wiki/xacro">
   <xacro:macro name="mobile_base_gazebo_plugin">
-    <gazebo>
-      <!-- ========== Diff Drive ========== -->
-      <plugin
-        filename="libgz-sim-diff-drive-system.so"
-        name="gz::sim::systems::DiffDrive">
-        <left_joint>left_wheel_joint</left_joint>
-        <right_joint>right_wheel_joint</right_joint>
-        <wheel_separation>0.26</wheel_separation>
-        <wheel_radius>0.04</wheel_radius>
-        <max_linear_velocity>0.5</max_linear_velocity>
-        <min_linear_velocity>-0.5</min_linear_velocity>
-        <max_angular_velocity>1.0</max_angular_velocity>
-        <min_angular_velocity>-1.0</min_angular_velocity>
-        <!-- ★ 使用绝对 topic -->
-        <topic>/cmd_vel</topic>
-        <odom_topic>/odom</odom_topic>
-        <tf_topic>/tf</tf_topic>
-        <frame_id>odom</frame_id>
-        <child_frame_id>base_link</child_frame_id>
-        <odom_publish_frequency>30</odom_publish_frequency>
-      </plugin>
-      <!-- ========== Joint States ========== -->
-      <plugin
-        filename="libgz-sim-joint-state-publisher-system.so"
-        name="gz::sim::systems::JointStatePublisher">
-        <topic>/joint_states</topic>
-      </plugin>
-      <!-- ========== Sensors ========== -->
-      <plugin
-        filename="libgz-sim-sensors-system.so"
-        name="gz::sim::systems::Sensors">
-        <render_engine>ogre2</render_engine>
-      </plugin>
-    </gazebo>
-  </xacro:macro>
+  <gazebo>
+    <plugin
+      filename="libignition-gazebo-diff-drive-system.so"
+      name="ignition::gazebo::systems::DiffDrive">
+      <left_joint>left_wheel_joint</left_joint>
+      <right_joint>right_wheel_joint</right_joint>
+      <wheel_separation>0.26</wheel_separation>
+      <wheel_radius>0.04</wheel_radius>
+      <max_linear_velocity>0.5</max_linear_velocity>
+      <min_linear_velocity>-0.5</min_linear_velocity>
+      <max_angular_velocity>1.0</max_angular_velocity>
+      <min_angular_velocity>-1.0</min_angular_velocity>
+      <topic>/cmd_vel</topic>
+      <odom_topic>/odom</odom_topic>
+      <tf_topic>/tf</tf_topic>
+      <frame_id>odom</frame_id>
+      <child_frame_id>base_footprint</child_frame_id>
+      <odom_publish_frequency>100</odom_publish_frequency>
+    </plugin>
+    <plugin
+      filename="libignition-gazebo-joint-state-publisher-system.so"
+      name="ignition::gazebo::systems::JointStatePublisher">
+      <topic>/joint_states</topic>
+      <update_rate>100</update_rate>
+    </plugin>
+    <plugin
+      filename="libignition-gazebo-sensors-system.so"
+      name="ignition::gazebo::systems::Sensors">
+      <render_engine>ogre2</render_engine>
+    </plugin>
+  </gazebo>
+</xacro:macro>
 </robot>

File: my_robot_description/urdf/sensors/lidar.xacro (robot description, xacro)
@@ -1,7 +1,5 @@
 <?xml version="1.0"?>
 <robot xmlns:xacro="http://www.ros.org/wiki/xacro">
-  <!-- ==================== 激光雷达 ==================== -->
   <xacro:macro name="lidar_sensor" params="prefix:='lidar'">
-    <!-- 激光雷达连杆 -->
     <link name="${prefix}_link">
       <visual>
@@ -10,5 +8,5 @@
           <cylinder length="0.05" radius="0.05"/>
         </geometry>
-        <material name="black"/>  <!-- 改为黑色，与底盘一致 -->
+        <material name="black"/>
       </visual>
       <collision>
@@ -20,14 +18,13 @@
       <xacro:cylinder_inertia m="0.1" r="0.05" h="0.05"/>
     </link>
-    <!-- 关节 - 安装在底盘上 -->
     <joint name="${prefix}_joint" type="fixed">
       <parent link="base_link"/>
       <child link="${prefix}_link"/>
-      <origin xyz="0 0 0.20" rpy="0 0 0"/>  <!-- 提高到0.20，避免碰撞 -->
+      <origin xyz="0.20 0 0.01" rpy="0 0 0"/>
     </joint>
-    <!-- Gazebo 插件：激光雷达 -->
     <gazebo reference="${prefix}_link">
-      <sensor name="${prefix}" type="ray">
-        <topic>scan</topic>
+      <sensor name="${prefix}" type="gpu_lidar">
+        <topic>/scan</topic>
+        <frame_id>${prefix}_link</frame_id>
         <pose>0 0 0 0 0 0</pose>
         <visualize>false</visualize>
@@ -48,5 +45,5 @@
           </range>
         </ray>
-        </sensor>
+      </sensor>
     </gazebo>
   </xacro:macro>
