Commit message: Add files via upload

File: my_robot_description/urdf/base/mobile_base.xacro (robot description, xacro)
@@ -1,89 +1,120 @@
 <?xml version="1.0"?>
 <robot xmlns:xacro="http://www.ros.org/wiki/xacro">
-    <xacro:macro name="mobile_base">
-        <xacro:property name="chassis_radius" value="0.14" /> <xacro:property name="chassis_height" value="0.12" />
-        <xacro:property name="chassis_mass" value="10.0" />   <xacro:property name="wheel_radius" value="0.04" />   <xacro:property name="wheel_width" value="0.02" />
-        <xacro:property name="wheel_offset_y" value="0.13" /> <xacro:property name="caster_radius" value="0.02" />  <xacro:property name="caster_offset_x" value="0.10" /> <material name="blue">
-            <color rgba="0.1 0.1 0.8 1"/>
-        </material>
-        <material name="black">
-            <color rgba="0.1 0.1 0.1 1"/>
-        </material>
-        <link name="base_footprint" />
-        <joint name="base_joint" type="fixed">
-            <parent link="base_footprint" />
-            <child link="base_link" />
-            <origin xyz="0 0 ${wheel_radius}" rpy="0 0 0" />
-        </joint>
-        <link name="base_link">
-            <visual>
-                <origin xyz="0 0 ${chassis_height/2}" rpy="0 0 0" />
-                <geometry>
-                    <cylinder radius="${chassis_radius}" length="${chassis_height}" />
-                </geometry>
-                <material name="blue" />
-            </visual>
-            <collision>
-                <origin xyz="0 0 ${chassis_height/2}" rpy="0 0 0" />
-                <geometry>
-                    <cylinder radius="${chassis_radius}" length="${chassis_height}" />
-                </geometry>
-            </collision>
-            <xacro:cylinder_inertia m="${chassis_mass}" r="${chassis_radius}" h="${chassis_height}" />
-        </link>
-        <xacro:macro name="wheel" params="prefix y_reflect">
-            <link name="${prefix}_wheel_link">
-                <visual>
-                    <origin xyz="0 0 0" rpy="${pi/2} 0 0" />
-                    <geometry>
-                        <cylinder radius="${wheel_radius}" length="${wheel_width}" />
-                    </geometry>
-                    <material name="black" />
-                </visual>
-                <collision>
-                    <origin xyz="0 0 0" rpy="${pi/2} 0 0" />
-                    <geometry>
-                        <cylinder radius="${wheel_radius}" length="${wheel_width}" />
-                    </geometry>
-                </collision>
-                <xacro:cylinder_inertia m="0.5" r="${wheel_radius}" h="${wheel_width}" />
-            </link>
-            <joint name="${prefix}_wheel_joint" type="continuous">
-                <parent link="base_link" />
-                <child link="${prefix}_wheel_link" />
-                <origin xyz="0 ${y_reflect * wheel_offset_y} 0" rpy="0 0 0" />
-                <axis xyz="0 1 0" />
-            </joint>
-        </xacro:macro>
-        <xacro:wheel prefix="left" y_reflect="1" />
-        <xacro:wheel prefix="right" y_reflect="-1" />
-        <xacro:macro name="caster_wheel" params="prefix x_reflect">
-            <link name="${prefix}_caster_wheel">
-                <visual>
-                    <geometry>
-                        <sphere radius="${caster_radius}" />
-                    </geometry>
-                    <material name="black" />
-                </visual>
-                <collision>
-                    <geometry>
-                        <sphere radius="${caster_radius}" />
-                    </geometry>
-                </collision>
-                <xacro:sphere_inertia m="0.1" r="${caster_radius}" />
-            </link>
-            <joint name="${prefix}_caster_joint" type="fixed">
-                <parent link="base_link" />
-                <child link="${prefix}_caster_wheel" />
-                <origin xyz="${x_reflect * caster_offset_x} 0 ${caster_radius - wheel_radius}" rpy="0 0 0" />
-            </joint>
-            <gazebo reference="${prefix}_caster_wheel">
-                <mu1>0.001</mu1>
-                <mu2>0.001</mu2>
-                <material>Gazebo/Black</material>
-            </gazebo>
-        </xacro:macro>
-        <xacro:caster_wheel prefix="front" x_reflect="1" />
-        <xacro:caster_wheel prefix="back" x_reflect="-1" />
+  <xacro:macro name="mobile_base">
+    <!-- ========== 参数 ========== -->
+    <xacro:property name="chassis_radius" value="0.14" />
+    <xacro:property name="chassis_height" value="0.12" />
+    <xacro:property name="chassis_mass" value="10.0" />
+    <xacro:property name="wheel_radius" value="0.04" />
+    <xacro:property name="wheel_width" value="0.02" />
+    <xacro:property name="wheel_offset_y" value="0.13" />
+    <xacro:property name="caster_radius" value="0.02" />
+    <xacro:property name="caster_offset_x" value="0.10" />
+    <!-- ========== base footprint ========== -->
+    <link name="base_footprint">
+    </link>
+    <joint name="base_joint" type="fixed">
+      <parent link="base_footprint"/>
+      <child link="base_link"/>
+      <origin xyz="0 0 ${wheel_radius}" rpy="0 0 0"/>
+    </joint>
+    <!-- ========== base link ========== -->
+    <link name="base_link">
+      <visual>
+        <origin xyz="0 0 ${chassis_height/2}" rpy="0 0 0"/>
+        <geometry>
+          <cylinder radius="${chassis_radius}" length="${chassis_height}"/>
+        </geometry>
+        <material name="blue"/>
+      </visual>
+      <collision>
+        <origin xyz="0 0 ${chassis_height/2}" rpy="0 0 0"/>
+        <geometry>
+          <cylinder radius="${chassis_radius}" length="${chassis_height}"/>
+        </geometry>
+      </collision>
+      <xacro:cylinder_inertia
+        m="${chassis_mass}"
+        r="${chassis_radius}"
+        h="${chassis_height}"/>
+    </link>
+    <!-- ========== 轮子宏 ========== -->
+    <xacro:macro name="wheel" params="prefix y_reflect">
+      <link name="${prefix}_wheel_link">
+        <visual>
+          <!-- 轮子横放 -->
+          <origin xyz="0 0 0" rpy="${pi/2} 0 0"/>
+          <geometry>
+            <cylinder radius="${wheel_radius}" length="${wheel_width}"/>
+          </geometry>
+          <material name="black"/>
+        </visual>
+        <collision>
+          <origin xyz="0 0 0" rpy="${pi/2} 0 0"/>
+          <geometry>
+            <cylinder radius="${wheel_radius}" length="${wheel_width}"/>
+          </geometry>
+        </collision>
+        <!-- ★★★ 关键修改：惯性矩阵的轴要与轮一致 ★★★ -->
+        <inertial>
+          <origin xyz="0 0 0" rpy="${pi/2} 0 0"/>
+          <mass value="0.5"/>
+          <inertia
+            ixx="${(0.5/12) * (3*wheel_radius*wheel_radius + wheel_width*wheel_width)}"
+            ixy="0" ixz="0"
+            iyy="${(0.5/12) * (3*wheel_radius*wheel_radius + wheel_width*wheel_width)}"
+            iyz="0"
+            izz="${(0.5/2) * (wheel_radius*wheel_radius)}"/>
+        </inertial>
+      </link>
+      <!-- ★★★ 关键修改：axis 改为   轴 ★★★ -->
+      <joint name="${prefix}_wheel_joint" type="continuous">
+        <parent link="base_link"/>
+        <child link="${prefix}_wheel_link"/>
+        <origin xyz="0 ${y_reflect * wheel_offset_y} 0" rpy="0 0 0"/>
+        <axis xyz="0 1 0"/>
+        <limit effort="0.2" velocity="20.0"/>
+      </joint>
+      <gazebo reference="${prefix}_wheel_link">
+        <mu1>1.0</mu1>
+        <mu2>1.0</mu2>
+        <kp>1000000.0</kp>
+        <kd>100.0</kd>
+        <gravity>true</gravity>
+        <self_collide>false</self_collide>
+      </gazebo>
     </xacro:macro>
+    <!-- 左右轮 -->
+    <xacro:wheel prefix="left"  y_reflect="1"/>
+    <xacro:wheel prefix="right" y_reflect="-1"/>
+    <!-- ========== 脚轮 ========== -->
+    <xacro:macro name="caster_wheel" params="prefix x_reflect">
+      <link name="${prefix}_caster_wheel">
+        <visual>
+          <geometry>
+            <sphere radius="${caster_radius}"/>
+          </geometry>
+          <material name="black"/>
+        </visual>
+        <collision>
+          <geometry>
+            <sphere radius="${caster_radius}"/>
+          </geometry>
+        </collision>
+        <xacro:sphere_inertia m="0.1" r="${caster_radius}"/>
+      </link>
+      <joint name="${prefix}_caster_joint" type="fixed">
+        <parent link="base_link"/>
+        <child link="${prefix}_caster_wheel"/>
+        <origin xyz="${x_reflect * caster_offset_x} 0 ${caster_radius - wheel_radius}" rpy="0 0 0"/>
+      </joint>
+      <gazebo reference="${prefix}_caster_wheel">
+        <mu1>0.001</mu1>
+        <mu2>0.001</mu2>
+        <gravity>true</gravity>
+      </gazebo>
+    </xacro:macro>
+    <xacro:caster_wheel prefix="front" x_reflect="1"/>
+    <xacro:caster_wheel prefix="back"  x_reflect="-1"/>
+  </xacro:macro>
 </robot>

File: my_robot_description/urdf/base/mobile_base_gazebo.xacro (robot description, xacro)
@@ -1,32 +1,36 @@
 <?xml version="1.0"?>
 <robot xmlns:xacro="http://www.ros.org/wiki/xacro">
-    <xacro:macro name="mobile_base_gazebo_plugin">
-        <gazebo>
-            <plugin filename="libignition-gazebo-diff-drive-system.so"
-                    name="ignition::gazebo::systems::DiffDrive">
-                <left_joint>left_wheel_joint</left_joint>
-                <right_joint>right_wheel_joint</right_joint>
-                <wheel_separation>0.26</wheel_separation>
-                <wheel_radius>0.04</wheel_radius>
-                <max_linear_acceleration>1</max_linear_acceleration>
-                <min_linear_acceleration>-1</min_linear_acceleration>
-                <max_angular_acceleration>2</max_angular_acceleration>
-                <min_angular_acceleration>-2</min_angular_acceleration>
-                <max_linear_velocity>0.5</max_linear_velocity>
-                <min_linear_velocity>-0.5</min_linear_velocity>
-                <max_angular_velocity>1</max_angular_velocity>
-                <min_angular_velocity>-1</min_angular_velocity>
-                <topic>cmd_vel</topic>
-                <odom_topic>odom</odom_topic>
-                <tf_topic>tf</tf_topic>
-                <frame_id>odom</frame_id>
-                <child_frame_id>base_footprint</child_frame_id>
-                <odom_publish_frequency>30</odom_publish_frequency>
-            </plugin>
-            <plugin filename="libignition-gazebo-joint-state-publisher-system.so"
-                    name="ignition::gazebo::systems::JointStatePublisher">
-                <topic>joint_states</topic>
-            </plugin>
-        </gazebo>
-    </xacro:macro>
+  <xacro:macro name="mobile_base_gazebo_plugin">
+  <gazebo>
+    <plugin
+      filename="libignition-gazebo-diff-drive-system.so"
+      name="ignition::gazebo::systems::DiffDrive">
+      <left_joint>left_wheel_joint</left_joint>
+      <right_joint>right_wheel_joint</right_joint>
+      <wheel_separation>0.26</wheel_separation>
+      <wheel_radius>0.04</wheel_radius>
+      <max_linear_velocity>0.5</max_linear_velocity>
+      <min_linear_velocity>-0.5</min_linear_velocity>
+      <max_angular_velocity>1.0</max_angular_velocity>
+      <min_angular_velocity>-1.0</min_angular_velocity>
+      <topic>/cmd_vel</topic>
+      <odom_topic>/odom</odom_topic>
+      <tf_topic>/tf</tf_topic>
+      <frame_id>odom</frame_id>
+      <child_frame_id>base_footprint</child_frame_id>
+      <odom_publish_frequency>100</odom_publish_frequency>
+    </plugin>
+    <plugin
+      filename="libignition-gazebo-joint-state-publisher-system.so"
+      name="ignition::gazebo::systems::JointStatePublisher">
+      <topic>/joint_states</topic>
+      <update_rate>100</update_rate>
+    </plugin>
+    <plugin
+      filename="libignition-gazebo-sensors-system.so"
+      name="ignition::gazebo::systems::Sensors">
+      <render_engine>ogre2</render_engine>
+    </plugin>
+  </gazebo>
+</xacro:macro>
 </robot>

File: my_robot_description/urdf/sensors/camera.xacro (robot description, xacro)
@@ -28,6 +28,6 @@
     <!-- Gazebo 插件：深度相机 -->
     <gazebo reference="${prefix}_link">
-      <material>Gazebo/Black</material>
       <sensor name="${prefix}" type="camera">
+        <topic>${prefix}/image_raw</topic>
         <camera>
           <horizontal_fov>1.0472</horizontal_fov>
@@ -44,10 +44,5 @@
         <always_on>true</always_on>
         <update_rate>30.0</update_rate>
-        <plugin filename="libignition-gazebo-camera-system.so"
-                name="ignition::gazebo::systems::Camera">
-          <topic>${prefix}/image_raw</topic>
-          <frame_id>${prefix}_link</frame_id>
-        </plugin>
-      </sensor>
+        </sensor>
     </gazebo>
   </xacro:macro>

File: my_robot_description/urdf/sensors/lidar.xacro (robot description, xacro)
@@ -1,33 +1,30 @@
 <?xml version="1.0"?>
 <robot xmlns:xacro="http://www.ros.org/wiki/xacro">
-  <!-- ==================== 激光雷达 ==================== -->
   <xacro:macro name="lidar_sensor" params="prefix:='lidar'">
-    <!-- 激光雷达连杆 -->
     <link name="${prefix}_link">
       <visual>
         <origin xyz="0 0 0" rpy="0 0 0"/>
         <geometry>
-          <cylinder length="0.05" radius="0.05"/>
+          <cylinder length="0.01" radius="0.01"/>
         </geometry>
-        <material name="black"/>  <!-- 改为黑色，与底盘一致 -->
+        <material name="black"/>
       </visual>
       <collision>
         <origin xyz="0 0 0" rpy="0 0 0"/>
         <geometry>
-          <cylinder length="0.05" radius="0.05"/>
+          <cylinder length="0.01" radius="0.01"/>
         </geometry>
       </collision>
       <xacro:cylinder_inertia m="0.1" r="0.05" h="0.05"/>
     </link>
-    <!-- 关节 - 安装在底盘上 -->
     <joint name="${prefix}_joint" type="fixed">
       <parent link="base_link"/>
       <child link="${prefix}_link"/>
-      <origin xyz="0 0 0.20" rpy="0 0 0"/>  <!-- 提高到0.20，避免碰撞 -->
+      <origin xyz="0.15 0 0.01" rpy="0 0 0"/>
     </joint>
-    <!-- Gazebo 插件：激光雷达 -->
     <gazebo reference="${prefix}_link">
-      <material>Gazebo/Black</material>
-      <sensor name="${prefix}" type="ray">
+      <sensor name="${prefix}" type="gpu_lidar">
+        <topic>/scan</topic>
+        <frame_id>${prefix}_link</frame_id>
         <pose>0 0 0 0 0 0</pose>
         <visualize>false</visualize>
@@ -36,5 +33,5 @@
           <scan>
             <horizontal>
-              <samples>360</samples>
+              <samples>720</samples>
               <resolution>1.0</resolution>
               <min_angle>-3.14159</min_angle>
@@ -43,14 +40,9 @@
           </scan>
           <range>
-            <min>0.1</min>
+            <min>0.2</min>
             <max>10.0</max>
             <resolution>0.01</resolution>
           </range>
         </ray>
-        <plugin filename="libignition-gazebo-raysensor-system.so"
-                name="ignition::gazebo::systems::RaySensor">
-          <topic>scan</topic>
-          <frame_id>${prefix}_link</frame_id>
-        </plugin>
       </sensor>
     </gazebo>
